File: power.kicad_sch (KiCad schematic)
At the start: 29 parts, among them Q1 DMP3099L-13, Q2 2N7002BK, U1 LP2985-10.0, U2 TLV74130P, U3 TLV74033P, U7 TPS62143

Commit message: replace U7 footprint vias by manually placed vias
The thermal vias in the footprint were being connected
to the groundplane with thermal reliefs and giving other
troubles (wrong drill size). This replaces them by manually
placed vias.

Signed-off-by: Daniel Estévez <daniel@destevez.net>
Parts:
- U7: footprint Package_DFN_QFN:VQFN-16-1EP_3x3mm_P0.5mm_EP1.68x1.68mm_ThermalVias -> Package_DFN_QFN:VQFN-16-1EP_3x3mm_P0.5mm_EP1.68x1.68mm
Changed lines of the file:
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@@
 			)
 		)
-		(property "Footprint" "Package_DFN_QFN:VQFN-16-1EP_3x3mm_P0.5mm_EP1.68x1.68mm_ThermalVias"
+		(property "Footprint" "Package_DFN_QFN:VQFN-16-1EP_3x3mm_P0.5mm_EP1.68x1.68mm"
 			(at 201.93 73.66 0)
 			(effects
